Commit message: fix: update max steering angle to 26° in configuration files and documentation

File: physicar_description/urdf/physicar_macros.xacro (robot description, xacro)
@@ -55,5 +55,5 @@
       <origin xyz="${x_offset} ${y_offset} 0" rpy="0 0 0"/>
       <axis xyz="0 0 1"/>
-      <limit lower="-0.5236" upper="0.5236" effort="25" velocity="1.0"/>
+      <limit lower="-0.4538" upper="0.4538" effort="25" velocity="1.0"/>
       <dynamics damping="0.1" friction="0.1"/>
     </joint>
