Commit message: Refactor code structure for improved readability and maintainability

File: physicar_description/urdf/physicar.urdf.xacro (robot description, xacro)
@@ -158,5 +158,5 @@
     <parent link="base_link"/>
     <child link="imu_link"/>
-    <origin xyz="0 0 0.05" rpy="0 0 0"/>
+    <origin xyz="0 0 0.0275" rpy="0 0 0"/>  <!-- 6.5cm from floor (base_link is at wheel_radius=3.75cm) -->
   </joint>
   <!-- ========== REAR WHEELS (Passive) ========== -->

Commit message: refactor: remove emergency stop, implement reverse brake, pan/tilt 45→30°, fix battery display
- Remove emergency stop system (LiDAR-based) from driver, servo controller,
  webserver UI/API, calibration endpoints, interfaces, and README docs
- Implement reverse brake with feedback loop (BRAKE_SPEED=0.3 m/s)
- Change pan/tilt max angle from 45° to 30° across all code, config, URDF,
  UI, joystick mapping, deepracer, and agent modules
- Fix steering URDF joint limit to match MAX_STEERING=20° (0.3491 rad)
- Fix battery display crash (restore missing parameter declarations)
- Remove emergency UI toggle from index.html and kiosk.html

File: physicar_description/urdf/physicar.urdf.xacro (robot description, xacro)
@@ -102,5 +102,5 @@
     <origin xyz="0.05 0.0 0.1" rpy="0 0 0"/>
     <axis xyz="0 0 1"/>
-    <limit lower="-0.7854" upper="0.7854" effort="10" velocity="1.0"/>
+    <limit lower="-0.5236" upper="0.5236" effort="10" velocity="1.0"/>
     <dynamics damping="0.1" friction="0.1"/>
   </joint>
@@ -130,5 +130,5 @@
     <origin xyz="0.025 0.0 0.013" rpy="0 0 0"/>
     <axis xyz="0 1 0"/>
-    <limit lower="-0.7854" upper="0.7854" effort="10" velocity="1.0"/>
+    <limit lower="-0.5236" upper="0.5236" effort="10" velocity="1.0"/>
     <dynamics damping="0.1" friction="0.1"/>
   </joint>

File: physicar_description/urdf/physicar_macros.xacro (robot description, xacro)
@@ -55,5 +55,5 @@
       <origin xyz="${x_offset} ${y_offset} 0" rpy="0 0 0"/>
       <axis xyz="0 0 1"/>
-      <limit lower="-0.4538" upper="0.4538" effort="25" velocity="1.0"/>
+      <limit lower="-0.3491" upper="0.3491" effort="25" velocity="1.0"/>
       <dynamics damping="0.1" friction="0.1"/>
     </joint>
